Commit message: occlusion progress

File: samk/automatic_annotator/urdf/_l515_annotation.urdf.xacro (robot description, xacro)
@@ -58,5 +58,5 @@
 	        <mesh filename="package://realsense2_description/meshes/l515.dae" />
         </geometry>
-      </xacro:if>
+    </xacro:if>
       </visual>
       <collision>
@@ -219,5 +219,5 @@
   </gazebo>
   <gazebo>
-    <plugin name="${name}_realsense_plugin" filename="librealsense_gazebo_plugin.so">
+    <plugin name="realsense_plugin" filename="librealsense_gazebo_plugin.so">
       <depthUpdateRate>6.0</depthUpdateRate>
       <colorUpdateRate>6.0</colorUpdateRate>

File: samk/automatic_annotator/urdf/samk_l515.urdf.xacro (robot description, xacro)
@@ -12,5 +12,5 @@
   </xacro:sensor_l515>
   <xacro:sensor_l515  parent="world" use_nominal_extrinsics="true" name="camera2" visible="false">
-    <origin xyz="1.5 1 1.5" rpy="0 1 3.14"/>
+    <origin xyz="0 0 1.5" rpy="0 0 0"/>
   </xacro:sensor_l515>
 </robot>
