Commit message: a lot of changes

File: samk/automatic_annotator/models/ball.urdf (robot description, URDF)
Before this commit: robot cube, 1 links, 0 joints
Links:
- link base_link: mass 0.0001 -> 0.1; geometry collision sphere radius=0.1; visual sphere radius=0.1

File: samk/automatic_annotator/urdf/samk_l515.urdf.xacro (robot description, xacro)
@@ -12,23 +12,29 @@
   </xacro:sensor_l515>
   <xacro:sensor_l515  parent="world" use_nominal_extrinsics="true" name="camera2" visible="false">
-    <origin xyz="1 0 1.5" rpy="0 1.57 0"/>
+    <origin xyz="0.8 0 1.5" rpy="0 1.57 0"/>
   </xacro:sensor_l515>
-  <xacro:sensor_l515  parent="world" use_nominal_extrinsics="true" name="camera3" visible="true">
-    <origin xyz="1.5 0.2 1.5" rpy="0 1.57 0"/>
+  <xacro:sensor_l515  parent="world" use_nominal_extrinsics="true" name="camera3" visible="false">
+    <origin xyz="0.6 1.5 0.3" rpy="0 0 -1.57"/>
   </xacro:sensor_l515>
-  <xacro:sensor_l515  parent="world" use_nominal_extrinsics="true" name="camera4" visible="true">
-    <origin xyz="1.5 0.2 1.5" rpy="0 1.57 0"/>
+  <xacro:sensor_l515  parent="world" use_nominal_extrinsics="true" name="camera4" visible="false">
+    <origin xyz="0.6 -1.5 0.3" rpy="0 0 1.57"/>
   </xacro:sensor_l515>
-  <xacro:sensor_l515  parent="world" use_nominal_extrinsics="true" name="camera5" visible="true">
-    <origin xyz="1.5 0.2 1.5" rpy="0 1.57 0"/>
+  <xacro:sensor_l515  parent="world" use_nominal_extrinsics="true" name="camera5" visible="false">
+    <origin xyz="1.4 1.4 1.5" rpy="0 1 -2.356"/>
   </xacro:sensor_l515>
-  <xacro:sensor_l515  parent="world" use_nominal_extrinsics="true" name="camera6" visible="true">
-    <origin xyz="1.5 0.2 1.5" rpy="0 1.57 0"/>
+  <xacro:sensor_l515  parent="world" use_nominal_extrinsics="true" name="camera6" visible="false">
+    <origin xyz="1.5 -1.3 1" rpy="0 0.8 2.356"/>
   </xacro:sensor_l515>
-  <xacro:sensor_l515  parent="world" use_nominal_extrinsics="true" name="camera7" visible="true">
-    <origin xyz="1.5 0.2 1.5" rpy="0 1.57 0"/>
+  <xacro:sensor_l515  parent="world" use_nominal_extrinsics="true" name="camera7" visible="false">
+    <origin xyz="-1 -1 1" rpy="0 0.3 0.6"/>
   </xacro:sensor_l515>
-  <xacro:sensor_l515  parent="world" use_nominal_extrinsics="true" name="camera8" visible="true">
-    <origin xyz="1.5 0.2 1.5" rpy="0 1.57 0"/>
+  <xacro:sensor_l515  parent="world" use_nominal_extrinsics="true" name="camera8" visible="false">
+    <origin xyz="2.5 0 0.5" rpy="0 0 3.14"/>
+  </xacro:sensor_l515>
+  <xacro:sensor_l515  parent="world" use_nominal_extrinsics="true" name="camera9" visible="false">
+    <origin xyz="0 -0.3 1.7" rpy="-0.8 1.37 1.03"/>
+  </xacro:sensor_l515>
+  <xacro:sensor_l515  parent="world" use_nominal_extrinsics="true" name="camera10" visible="false">
+    <origin xyz="-1 1 0.7" rpy="0 0.3 -0.6"/>
   </xacro:sensor_l515>
 </robot>
