Commit message: ready for testing

File: samk/automatic_annotator/models/big_ball.urdf (robot description, URDF)
Before this commit: robot ball, 1 links, 0 joints
Links:
- link base_link: geometry collision sphere radius=0.3; visual sphere radius=0.3

File: samk/automatic_annotator/models/box.urdf (robot description, URDF)
Before this commit: robot cube, 1 links, 0 joints
Links:
- link base_link: mass 0.0001 -> 0.00001; geometry collision box size=0.05 0.05 0.05; visual box size=0.05 0.05 0.05

File: samk/automatic_annotator/models/rectangle.urdf (robot description, URDF)
Before this commit: robot ball, 1 links, 0 joints
Links:
- link base_link: geometry collision box size=0.1 0.1 0.01; visual box size=0.1 0.1 0.01

File: samk/automatic_annotator/urdf/_l515_annotation.urdf.xacro (robot description, xacro)
@@ -220,7 +220,7 @@
   <gazebo>
     <plugin name="realsense_plugin" filename="librealsense_gazebo_plugin.so">
-      <depthUpdateRate>6.0</depthUpdateRate>
-      <colorUpdateRate>6.0</colorUpdateRate>
-      <infraredUpdateRate>6.0</infraredUpdateRate>
+      <depthUpdateRate>60.0</depthUpdateRate>
+      <colorUpdateRate>60.0</colorUpdateRate>
+      <infraredUpdateRate>60.0</infraredUpdateRate>
       <depthTopicName>${name}_depth/image_raw</depthTopicName>
       <depthCameraInfoTopicName>${name}_depth/camera_info</depthCameraInfoTopicName>
